File: board/fontes_alimentacao.kicad_sch (KiCad schematic)
At the start: 4 parts, among them J1 Conn_02x02_Top_Bottom, U50 YAAJ_DCDC_StepDown_LM2596

Commit message: Schematic changes and board creation
Parts:
- F1: value Polyfuse -> 1.85A
- F2: value Polyfuse -> 3A
- renumbered J1 to J2, U50 to U3
Connections:
- net GND_micro is gone; now on net GND: U3.3 (GND)
- net +12V: now reaches F1.1, J2.3 (Pin_3)
- net +12V: now also J2.1 (Pin_1)
- net GND: now reaches J2.2 (Pin_2)
- net GND: now also J2.4 (Pin_4), U3.2 (GND)
Other:
- moved on the sheet: F1, F2, J2, U3
