File: board/RC_filter.kicad_sch (KiCad schematic)
At the start: 2 parts

Commit message: Criação da placa de alimentação
Other:
- company: (none) -> Escola Politécnica da Universidade de São Paulo
Changed lines of the file:
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@@
 	(generator_version "8.0")
 	(paper "A4")
+	(title_block
+		(date "2025-10-02")
+		(company "Escola Politécnica da Universidade de São Paulo")
+	)
 	(junction
 		(at 97.79 93.98)
