File: board/board.kicad_pcb (KiCad board)
At the start: 2 copper layers, 327.2 x 141.6 mm, 138 parts, among them J1 Conn_01x03_Pin, J10 Conn_02x07_Odd_Even, J11 Conn_01x02_Pin, J12 Conn_01x02_Pin, J13 Conn_02x07_Odd_Even, J14 Conn_01x02_Pin, J15 Conn_01x02_Pin, J16 Conn_02x07_Odd_Even, J17 Conn_01x02_Pin, J18 Conn_01x02_Pin, J2 Conn_01x02_Pin, J3 Conn_01x02_Pin, J4 Conn_02x02_ZigZag, J5 Conn_02x03_ZigZag, J6 Conn_02x02_ZigZag, J7 Conn_01x03_Pin, J8 Conn_01x03_Pin, J9 Conn_01x03_Pin, U1 ESP32-DevKitC, U10 H11L1, U11 H11L1, U12 H11L1, U13 HEF4093B, U14 H11L1, U15 H11L1, U16 H11L1, U17 HEF4093B, U18 H11L1, U19 H11L1, U2 LM324, U20 H11L1, U3 LV25-P, U4 LV25-P, U5 LM324, U6 LM324, U7 LM324, U8 LM324, U9 HEF4093B

Commit message: Finalização da placa, trilhas, planos de terra e footprint TJA1050
Parts:
- removed the U1 at (85.4, 82.2)
- added C35: 0,1u, Capacitor_THT:C_Disc_D8.0mm_W5.0mm_P7.50mm, F.Cu at (62.1, 129.5)
- added C36: 0,1u, Capacitor_THT:C_Disc_D8.0mm_W5.0mm_P7.50mm, F.Cu at (82.4, 122.3)
- added C37: 0,1u, Capacitor_THT:C_Disc_D8.0mm_W5.0mm_P7.50mm, F.Cu at (71.8, 122.1)
- added J19: Conn_02x02_ZigZag, Connector_Molex:Molex_Mini-Fit_Jr_5566-04A_2x02_P4.20mm_Vertical, F.Cu at (49.2, 148.5)
- added U17: ESP32-DevKitC, Espressif:ESP32-DevKitC, F.Cu at (87.8, 76.5)
- added U18: ~, Modules:TJA1050, F.Cu at (64.0, 132.9)
- added U19: ESP32-DevKitC, Espressif:ESP32-DevKitC, F.Cu at (112.7, 129.9)
- moved R36 74.2 mm to (47.0, 124.5)
- moved J9 65.5 mm to (27.8, 120.9), turned to 90 degrees
- moved R37 62.6 mm to (49.3, 121.3)
- moved R40 62.6 mm to (56.9, 124.5)
- moved C13 60.0 mm to (34.5, 118.4)
- moved R34 60.0 mm to (58.2, 108.0)
- moved R35 60.0 mm to (48.3, 108.0)
- moved R38 60.0 mm to (58.0, 118.5)
- moved R39 60.0 mm to (51.7, 121.3)
- moved U7 60.0 mm to (39.0, 118.5)
- moved C28 58.0 mm to (161.9, 41.3), turned to 0 degrees
- moved C14 57.0 mm to (161.8, 83.7), turned to 0 degrees
- moved C21 56.3 mm to (161.7, 126.2), turned to 0 degrees
- moved J15 52.8 mm to (173.5, 147.2), turned to 180 degrees
- moved J18 52.7 mm to (173.7, 62.3), turned to 180 degrees
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- renumbered U2 to U1, U11 to U10, U12 to U11, U13 to U12, U14 to U13, U15 to U14, U16 to U15, U17 to U16, U3 to U2, U18 to U20, U19 to U21, U20 to U22, U4 to U3, U5 to U4, U6 to U5, U7 to U6, U8 to U7, U9 to U8, U10 to U9
Connections:
- C20 pad 1: +5V -> +3.3V
- C27 pad 1: +5V -> +3.3V
- C32 pad 1: +5V -> +3.3V
- R46 pad 1: +5V -> +3.3V
- R52 pad 1: +5V -> +3.3V
- R56 pad 1: +5V -> +3.3V
- U11 pad 6: +5V -> +3.3V
- U12 pad 1: unconnected-(U13-Pad1) -> /PWM - 15V Level Shifter/Conectores - PWM e erro2/Isolação de sinais - PWM7/output_sign
- U12 pad 11: unconnected-(U13-Pad11) -> /PWM - 15V Level Shifter/Conectores - PWM e erro2/PWM_TOP_driver
- U12 pad 12: unconnected-(U13-Pad12) -> /PWM - 15V Level Shifter/Conectores - PWM e erro2/Isolação de sinais - PWM7/output_sign
- U12 pad 13: unconnected-(U13-Pad13) -> /PWM - 15V Level Shifter/Conectores - PWM e erro2/Isolação de sinais - PWM7/output_sign
- U12 pad 2: unconnected-(U13-Pad2) -> /PWM - 15V Level Shifter/Conectores - PWM e erro2/Isolação de sinais - PWM7/output_sign
- U12 pad 4: /PWM - 15V Level Shifter/Conectores - PWM e erro2/PWM_TOP_driver -> unconnected-(U12-Pad4)
- U12 pad 5: /PWM - 15V Level Shifter/Conectores - PWM e erro2/Isolação de sinais - PWM7/output_sign -> /PWM - 15V Level Shifter/Conectores - PWM e erro2/Isolação de sinais - PWM6/output_sign
- U12 pad 6: /PWM - 15V Level Shifter/Conectores - PWM e erro2/Isolação de sinais - PWM7/output_sign -> /PWM - 15V Level Shifter/Conectores - PWM e erro2/Isolação de sinais - PWM6/output_sign
- U15 pad 6: +5V -> +3.3V
- U16 pad 1: unconnected-(U17-Pad1) -> /PWM - 15V Level Shifter/Conectores - PWM e erro/Isolação de sinais - PWM7/output_sign
- U16 pad 11: unconnected-(U17-Pad11) -> /PWM - 15V Level Shifter/Conectores - PWM e erro/PWM_TOP_driver
- U16 pad 12: unconnected-(U17-Pad12) -> /PWM - 15V Level Shifter/Conectores - PWM e erro/Isolação de sinais - PWM7/output_sign
- U16 pad 13: unconnected-(U17-Pad13) -> /PWM - 15V Level Shifter/Conectores - PWM e erro/Isolação de sinais - PWM7/output_sign
- U16 pad 2: unconnected-(U17-Pad2) -> /PWM - 15V Level Shifter/Conectores - PWM e erro/Isolação de sinais - PWM7/output_sign
- U16 pad 4: /PWM - 15V Level Shifter/Conectores - PWM e erro/PWM_TOP_driver -> unconnected-(U16-Pad4)
- U16 pad 5: /PWM - 15V Level Shifter/Conectores - PWM e erro/Isolação de sinais - PWM7/output_sign -> /PWM - 15V Level Shifter/Conectores - PWM e erro/Isolação de sinais - PWM6/output_sign
- U16 pad 6: /PWM - 15V Level Shifter/Conectores - PWM e erro/Isolação de sinais - PWM7/output_sign -> /PWM - 15V Level Shifter/Conectores - PWM e erro/Isolação de sinais - PWM6/output_sign
- U21 pad 6: +5V -> +3.3V
- U8 pad 1: unconnected-(U9-Pad1) -> /PWM - 15V Level Shifter/Conectores - PWM e erro1/Isolação de sinais - PWM7/output_sign
- U8 pad 11: unconnected-(U9-Pad11) -> /PWM - 15V Level Shifter/Conectores - PWM e erro1/PWM_TOP_driver
- U8 pad 12: unconnected-(U9-Pad12) -> /PWM - 15V Level Shifter/Conectores - PWM e erro1/Isolação de sinais - PWM7/output_sign
- U8 pad 13: unconnected-(U9-Pad13) -> /PWM - 15V Level Shifter/Conectores - PWM e erro1/Isolação de sinais - PWM7/output_sign
- U8 pad 2: unconnected-(U9-Pad2) -> /PWM - 15V Level Shifter/Conectores - PWM e erro1/Isolação de sinais - PWM7/output_sign
- U8 pad 4: /PWM - 15V Level Shifter/Conectores - PWM e erro1/PWM_TOP_driver -> unconnected-(U8-Pad4)
- U8 pad 5: /PWM - 15V Level Shifter/Conectores - PWM e erro1/Isolação de sinais - PWM7/output_sign -> /PWM - 15V Level Shifter/Conectores - PWM e erro1/Isolação de sinais - PWM6/output_sign
- U8 pad 6: /PWM - 15V Level Shifter/Conectores - PWM e erro1/Isolação de sinais - PWM7/output_sign -> /PWM - 15V Level Shifter/Conectores - PWM e erro1/Isolação de sinais - PWM6/output_sign
Routing:
- net +3.3V: track 0.00 -> 277.5 mm
- net +15V: track 117.5 -> 339.8 mm, vias 0 -> 4
- net Vdrive: track 76.4 -> 273.8 mm
- net -15V: track 262.0 -> 357.1 mm, vias 0 -> 4
- net /MicroControladores/CS: track 0.00 -> 78.7 mm
- net /err_3: track 9.96 -> 72.6 mm
- net /PWM_BOT_3: track 4.67 -> 60.9 mm
- net GND1: track 0.00 -> 47.3 mm
- net /PWM_TOP_3: track 4.67 -> 51.2 mm
- net /MicroControladores/CAN_RX: track 0.00 -> 43.3 mm
- net /PWM_TOP_1: track 4.67 -> 45.0 mm
- net /Adequação Sinais Corrente e Tensão/Filtro RC5/unfilt_signal: track 6.18 -> 46.5 mm
- net /MicroControladores/SCK: track 0.00 -> 39.3 mm
- net /MicroControladores/CAN_TX: track 0.00 -> 34.9 mm
- net /PWM_BOT_1: track 4.67 -> 38.0 mm
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- added copper zone on B.Cu, net GND
- added copper zone on F.Cu, net GND
- added copper zone on B.Cu, net GND1
- added copper zone on F.Cu, net GND1
Other:
- board size 327.2 x 141.6 mm -> 170 x 150 mm

Commit message: Criação da placa de alimentação
Parts:
- added J20: Conn_01x02_Pin, Modules:Molex_Mini-Fit_Jr_5566-02A_2x01_P4.20mm_Vertical, F.Cu at (34.2, 132.8)
- J19: value Conn_02x02_ZigZag -> Conn_01x02_Pin; footprint Connector_Molex:Molex_Mini-Fit_Jr_5566-04A_2x02_P4.20mm_Vertical -> Modules:Molex_Mini-Fit_Jr_5566-02A_2x01_P4.20mm_Vertical
- J4, J6: footprint Connector_Molex:Molex_Mini-Fit_Jr_5566-04A_2x02_P4.20mm_Vertical -> Modules:Molex_Mini-Fit_Jr_5566-04A_2x02_P4.20mm_Vertical
- J5: footprint Connector_Molex:Molex_Mini-Fit_Jr_5566-06A_2x03_P4.20mm_Vertical -> Modules:Molex_Mini-Fit_Jr_5566-06A_2x03_P4.20mm_Vertical
- moved F1 29.1 mm to (48.6, 156.6), turned to 90 degrees
- moved J19 28.7 mm to (25.2, 132.8), turned to 0 degrees
- moved J4 20.6 mm to (55.2, 152.4), turned to 0 degrees
- moved RV2 16.7 mm to (48.6, 36.5), turned to 180 degrees
- moved J5 12.8 mm to (55.8, 30.5), turned to 180 degrees
- moved RV1 12.5 mm to (54.6, 146.3), turned to 0 degrees
- moved C29 8.45 mm to (68.7, 134.7), turned to -90 degrees
- moved U18 7.42 mm to (63.3, 140.3), turned to 180 degrees
- moved F2 5.05 mm to (42.6, 25.5)
- moved F3 5.05 mm to (62.0, 25.5)
- moved RV3 0.65 mm to (61.2, 36.5), turned to 180 degrees
- renumbered C35 to C29, C36 to C30, C37 to C31, C29 to C32, C30 to C33, C31 to C34, C32 to C35, C33 to C36, C34 to C37
Connections:
- J19 pad 1: /MicroControladores/CANH -> /MicroControladores/CANL
- J19 pad 2: /MicroControladores/CANL -> /MicroControladores/CANH
- J5 pad 1: /Power Connectors/+15V_sym_conn -> /Power Connectors/-15V_sym_conn
- J5 pad 3: /Power Connectors/-15V_sym_conn -> /Power Connectors/+15V_sym_conn
- J5 pad 4: /Power Connectors/+15V_sym_conn -> /Power Connectors/-15V_sym_conn
- J5 pad 6: /Power Connectors/-15V_sym_conn -> /Power Connectors/+15V_sym_conn
- U19 pad 10: /MicroControladores/CAN_RX -> /MicroControladores/CAN_TX
- U19 pad 11: /MicroControladores/CAN_TX -> /MicroControladores/CAN_RX
Routing:
- net +5V: track 55.7 -> 77.2 mm
- net +15V: track 339.8 -> 353.0 mm
- net /MicroControladores/CAN_RX: track 43.3 -> 32.2 mm
- net /MicroControladores/CANL: track 13.3 -> 18.6 mm
- net GND: track 5.97 -> 0.76 mm
- net -15V: track 357.1 -> 361.3 mm
- net /Power Connectors/+15V_sym_conn: track 14.8 -> 19.0 mm
- net /Power Connectors/-15V_sym_conn: track 16.3 -> 18.2 mm
- net /MicroControladores/CANH: track 17.5 -> 19.5 mm
- net /MicroControladores/CAN_TX: track 34.9 -> 36.5 mm
Other:
- board text added: "15V"
- board text added: "5V"
- board text added: "BOT"
- board text added: "CANH"
- board text added: "CANL"
- board text added: "TOP"
- board text added: "± 15V"
