File: board/micro_comm.kicad_sch (KiCad schematic)
At the start: 7 parts, among them J19 Conn_02x02_ZigZag, U17 ESP32-DevKitC, U19 ESP32-DevKitC

Commit message: Criação da placa de alimentação
Parts:
- removed J19: Conn_02x02_ZigZag, Connector_Molex:Molex_Mini-Fit_Jr_5566-04A_2x02_P4.20mm_Vertical, symbol Connectors:Conn_02x02_ZigZag
- added J19, J20: Conn_01x02_Pin, Modules:Molex_Mini-Fit_Jr_5566-02A_2x01_P4.20mm_Vertical, symbol Connector:Conn_01x02_Pin
- renumbered C35 to C29, C36 to C30, C37 to C31
Connections:
- net CANH: now also J19.2 (Pin_2), J20.2 (Pin_2)
- net CANL: now also J19.1 (Pin_1), J20.1 (Pin_1)
- net CAN_RX: now also U19.11 (ADC2_CH7/GPIO27); no longer U19.10 (DAC_2/ADC2_CH9/GPIO26)
- net CAN_TX: now also U19.10 (DAC_2/ADC2_CH9/GPIO26); no longer U19.11 (ADC2_CH7/GPIO27)
Other:
- company: (none) -> Escola Politécnica da Universidade de São Paulo
