File: board/pwr_conn.kicad_sch (KiCad schematic)
At the start: 11 parts, among them J4 Conn_02x02_ZigZag, J5 Conn_02x03_ZigZag, J6 Conn_02x02_ZigZag

Commit message: Criação da placa de alimentação
Parts:
- J4, J6: footprint Connector_Molex:Molex_Mini-Fit_Jr_5566-04A_2x02_P4.20mm_Vertical -> Modules:Molex_Mini-Fit_Jr_5566-04A_2x02_P4.20mm_Vertical
- J5: footprint Connector_Molex:Molex_Mini-Fit_Jr_5566-06A_2x03_P4.20mm_Vertical -> Modules:Molex_Mini-Fit_Jr_5566-06A_2x03_P4.20mm_Vertical
Connections:
- net +15V_sym_conn: now also J5.3 (Pin_3), J5.6 (Pin_6); no longer J5.1 (Pin_1), J5.4 (Pin_4)
- net -15V_sym_conn: now also J5.1 (Pin_1), J5.4 (Pin_4); no longer J5.3 (Pin_3), J5.6 (Pin_6)
Other:
- company: (none) -> Escola Politécnica da Universidade de São Paulo
Changed lines of the file:
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@@
 	(generator_version "8.0")
 	(paper "A4")
+	(title_block
+		(date "2025-10-02")
+		(company "Escola Politécnica da Universidade de São Paulo")
+	)
 	(junction
 		(at 81.28 62.23)
@@
 		)
 	)
+	(label "+15V_sym_conn"
+		(at 30.48 76.2 180)
+		(effects
+			(font
+				(size 1.27 1.27)
+			)
+			(justify right bottom)
+		)
+	)
 	(label "Vdrive"
 		(at 96.52 116.84 0)
@@
 		)
 	)
-	(label "+15V_sym_conn"
-		(at 43.18 71.12 0)
-		(effects
-			(font
-				(size 1.27 1.27)
-			)
-			(justify left bottom)
-		)
-	)
 	(label "5V_conn"
 		(at 30.48 30.48 180)
@@
 		)
 	)
-	(label "-15V_sym_conn"
-		(at 43.18 76.2 0)
-		(effects
-			(font
-				(size 1.27 1.27)
-			)
-			(justify left bottom)
-		)
-	)
 	(label "5V_conn"
 		(at 77.47 26.67 180)
@@
 	)
 	(label "+15V_sym_conn"
-		(at 30.48 71.12 180)
-		(effects
-			(font
-				(size 1.27 1.27)
-			)
-			(justify right bottom)
+		(at 43.18 76.2 0)
+		(effects
+			(font
+				(size 1.27 1.27)
+			)
+			(justify left bottom)
 		)
 	)
@@
 		)
 	)
+	(label "-15V_sym_conn"
+		(at 43.18 71.12 0)
+		(effects
+			(font
+				(size 1.27 1.27)
+			)
+			(justify left bottom)
+		)
+	)
 	(label "Vdrive_conn"
 		(at 78.74 116.84 180)
@@
 		)
 	)
-	(label "-15V_sym_conn"
-		(at 30.48 76.2 180)
-		(effects
-			(font
-				(size 1.27 1.27)
-			)
-			(justify right bottom)
-		)
-	)
 	(label "GND_sym"
 		(at 111.76 72.39 0)
@@
 			)
 			(justify left bottom)
+		)
+	)
+	(label "-15V_sym_conn"
+		(at 30.48 71.12 180)
+		(effects
+			(font
+				(size 1.27 1.27)
+			)
+			(justify right bottom)
 		)
 	)
@@
 			)
 		)
-		(property "Footprint" "Connector_Molex:Molex_Mini-Fit_Jr_5566-06A_2x03_P4.20mm_Vertical"
+		(property "Footprint" "Modules:Molex_Mini-Fit_Jr_5566-06A_2x03_P4.20mm_Vertical"
 			(at 35.56 73.66 0)
 			(effects
@@
 			)
 		)
-		(property "Footprint" "Connector_Molex:Molex_Mini-Fit_Jr_5566-04A_2x02_P4.20mm_Vertical"
+		(property "Footprint" "Modules:Molex_Mini-Fit_Jr_5566-04A_2x02_P4.20mm_Vertical"
 			(at 35.56 120.65 0)
 			(effects
@@
 			)
 		)
-		(property "Footprint" "Connector_Molex:Molex_Mini-Fit_Jr_5566-04A_2x02_P4.20mm_Vertical"
+		(property "Footprint" "Modules:Molex_Mini-Fit_Jr_5566-04A_2x02_P4.20mm_Vertical"
 			(at 35.56 30.48 0)
 			(effects
