File: Placas/Controle/Controle.kicad_pcb (KiCad board)
At the start: 2 copper layers, 170 x 150 mm, 145 parts, among them J1 Conn_02x03_ZigZag, J10 Conn_01x03_Pin, J11 Conn_01x02_Pin, J12 Conn_01x02_Pin, J13 Conn_02x07_Odd_Even, J14 Conn_01x02_Pin, J15 Conn_01x02_Pin, J16 Conn_01x03_Pin, J17 Conn_02x02_ZigZag, J18 Conn_01x02_Pin, J19 Conn_01x02_Pin, J2 Conn_01x02_Pin, J20 Conn_02x07_Odd_Even, J3 Conn_01x02_Pin, J4 Conn_02x02_ZigZag, J5 Conn_01x03_Pin, J6 Conn_01x02_Pin, J7 Conn_01x03_Pin, J8 Conn_01x02_Pin, J9 Conn_02x07_Odd_Even, U1 LV25-P, U10 H11L1, U11 H11L1, U12 LM324, U13 HEF4093B, U14 H11L1, U15 LM324, U16 ESP32-DevKitC, U17 H11L1, U18 HEF4093B, U19 H11L1, U2 LV25-P, U20 H11L1, U22 H11L1, U3 LM324, U4 LM324, U5 H11L1, U6 HEF4093B, U7 H11L1, U8 LM324, U9 ESP32-DevKitC

Commit message: Adição de circuitos opcionais para PWM
Parts:
- added C38: 0,1u, Capacitor_THT:C_Disc_D8.0mm_W5.0mm_P7.50mm, F.Cu at (426.0, 176.1)
- added C39: ${C_in}, Capacitor_THT:C_Disc_D8.0mm_W5.0mm_P7.50mm, F.Cu at (449.8, 141.5)
- added C40: 0,1u, Capacitor_THT:C_Disc_D8.0mm_W5.0mm_P7.50mm, F.Cu at (449.8, 148.1)
- added C41: ${C_in}, Capacitor_THT:C_Disc_D8.0mm_W5.0mm_P7.50mm, F.Cu at (449.8, 169.6)
- added C42: 0,1u, Capacitor_THT:C_Disc_D8.0mm_W5.0mm_P7.50mm, F.Cu at (449.8, 176.1)
- added C43: ${C_in}, Capacitor_THT:C_Disc_D8.0mm_W5.0mm_P7.50mm, F.Cu at (426.0, 141.5)
- added C44: 0,1u, Capacitor_THT:C_Disc_D8.0mm_W5.0mm_P7.50mm, F.Cu at (426.0, 148.1)
- added Q1: BC337, Package_TO_SOT_THT:TO-92_Inline, F.Cu at (439.3, 133.7)
- added Q2: BC337, Package_TO_SOT_THT:TO-92_Inline, F.Cu at (340.1, 164.0)
- added Q3: BC337, Package_TO_SOT_THT:TO-92_Inline, F.Cu at (439.4, 51.2)
- added Q4: BC337, Package_TO_SOT_THT:TO-92_Inline, F.Cu at (415.5, 133.7)
- added Q5: BC337, Package_TO_SOT_THT:TO-92_Inline, F.Cu at (439.3, 161.7)
- added Q6: BC337, Package_TO_SOT_THT:TO-92_Inline, F.Cu at (415.5, 161.7)
- added R59: ${R_out_pullup}, Resistor_THT:R_Axial_DIN0207_L6.3mm_D2.5mm_P7.62mm_Horizontal, F.Cu at (439.0, 46.0)
- added R60: ${R_in}, Resistor_THT:R_Axial_DIN0207_L6.3mm_D2.5mm_P7.62mm_Horizontal, F.Cu at (415.0, 112.2)
- added R61: ${R_in_bjt}, Resistor_THT:R_Axial_DIN0207_L6.3mm_D2.5mm_P7.62mm_Horizontal, F.Cu at (415.0, 116.3)
- added R62: ${R_base_emitter}, Resistor_THT:R_Axial_DIN0207_L6.3mm_D2.5mm_P7.62mm_Horizontal, F.Cu at (415.0, 120.3)
- added R63: ${R_pullup_bjt}, Resistor_THT:R_Axial_DIN0207_L6.3mm_D2.5mm_P7.62mm_Horizontal, F.Cu at (415.0, 124.4)
- added R64: ${R_out_pullup}, Resistor_THT:R_Axial_DIN0207_L6.3mm_D2.5mm_P7.62mm_Horizontal, F.Cu at (415.0, 128.4)
- added R65: ${R_in}, Resistor_THT:R_Axial_DIN0207_L6.3mm_D2.5mm_P7.62mm_Horizontal, F.Cu at (415.0, 168.3)
- added R66: ${R_1}, Resistor_THT:R_Axial_DIN0207_L6.3mm_D2.5mm_P7.62mm_Horizontal, F.Cu at (415.0, 172.4)
- added R67: ${R_2}, Resistor_THT:R_Axial_DIN0207_L6.3mm_D2.5mm_P7.62mm_Horizontal, F.Cu at (415.0, 176.4)
- added R68: ${R_out_pullup}, Resistor_THT:R_Axial_DIN0207_L6.3mm_D2.5mm_P7.62mm_Horizontal, F.Cu at (415.0, 180.5)
- added R69: ${R_in}, Resistor_THT:R_Axial_DIN0207_L6.3mm_D2.5mm_P7.62mm_Horizontal, F.Cu at (438.9, 140.3)
- added R70: ${R_in_bjt}, Resistor_THT:R_Axial_DIN0207_L6.3mm_D2.5mm_P7.62mm_Horizontal, F.Cu at (438.9, 144.3)
- added R71: ${R_base_emitter}, Resistor_THT:R_Axial_DIN0207_L6.3mm_D2.5mm_P7.62mm_Horizontal, F.Cu at (438.9, 148.4)
- added R72: ${R_pullup_bjt}, Resistor_THT:R_Axial_DIN0207_L6.3mm_D2.5mm_P7.62mm_Horizontal, F.Cu at (438.9, 152.4)
- added R73: ${R_out_pullup}, Resistor_THT:R_Axial_DIN0207_L6.3mm_D2.5mm_P7.62mm_Horizontal, F.Cu at (438.9, 156.5)
- added R74: ${R_in}, Resistor_THT:R_Axial_DIN0207_L6.3mm_D2.5mm_P7.62mm_Horizontal, F.Cu at (438.9, 168.3)
- added R75: ${R_1}, Resistor_THT:R_Axial_DIN0207_L6.3mm_D2.5mm_P7.62mm_Horizontal, F.Cu at (438.9, 172.4)
- added R76: ${R_2}, Resistor_THT:R_Axial_DIN0207_L6.3mm_D2.5mm_P7.62mm_Horizontal, F.Cu at (438.9, 176.4)
- added R77: ${R_out_pullup}, Resistor_THT:R_Axial_DIN0207_L6.3mm_D2.5mm_P7.62mm_Horizontal, F.Cu at (438.9, 180.5)
- added R78: ${R_in}, Resistor_THT:R_Axial_DIN0207_L6.3mm_D2.5mm_P7.62mm_Horizontal, F.Cu at (415.0, 140.3)
- added R79: ${R_in_bjt}, Resistor_THT:R_Axial_DIN0207_L6.3mm_D2.5mm_P7.62mm_Horizontal, F.Cu at (415.0, 144.3)
- added R80: ${R_base_emitter}, Resistor_THT:R_Axial_DIN0207_L6.3mm_D2.5mm_P7.62mm_Horizontal, F.Cu at (415.0, 148.4)
- added R81: ${R_pullup_bjt}, Resistor_THT:R_Axial_DIN0207_L6.3mm_D2.5mm_P7.62mm_Horizontal, F.Cu at (415.0, 152.4)
- added R82: ${R_out_pullup}, Resistor_THT:R_Axial_DIN0207_L6.3mm_D2.5mm_P7.62mm_Horizontal, F.Cu at (415.0, 156.5)
- added U23: H11L1, Package_DIP:DIP-6_W7.62mm, F.Cu at (449.7, 153.4)
- added U24: H11L1, Package_DIP:DIP-6_W7.62mm, F.Cu at (449.7, 181.5)
- added U25: H11L1, Package_DIP:DIP-6_W7.62mm, F.Cu at (425.9, 153.4)
- C1, C16, C17: footprint Capacitor_THT:C_Disc_D8.0mm_W5.0mm_P7.50mm -> Capacitor_SMD:C_0805_2012Metric_Pad1.18x1.45mm_HandSolder
- C10, C13, C14: value 0,1u -> 330n
- C15: value C_err -> 330n
- C18, C20: value 330n -> 10u; footprint Capacitor_THT:C_Disc_D8.0mm_W5.0mm_P7.50mm -> Capacitor_SMD:C_1210_3225Metric_Pad1.33x2.70mm_HandSolder
- C19: value 330n -> 0,1u; footprint Capacitor_THT:C_Disc_D8.0mm_W5.0mm_P7.50mm -> Capacitor_SMD:C_0805_2012Metric_Pad1.18x1.45mm_HandSolder
- C21: value 330n -> 0,1u
- C22, C23, C36, C6: value C_pwm -> 0,1u
- C25: value C_err -> 0,1u
- C27, C29, C33, C35: value 0,1u -> ${C_in}
- C3: value 0,1u -> 4,7u
- C31: value C_pwm -> ${C_in}
- C37: value C_err -> ${C_in}
- C5: value C_pwm -> 4,7u
- F1: value 0,4A -> 1A
- F3: value 3A -> 0,4A
- F4: value 1A -> 3A
- J1: value Conn_02x03_ZigZag -> Conn_02x02; footprint Modules:Molex_Mini-Fit_Jr_5566-06A_2x03_P4.20mm_Vertical -> Minifit:Molex_Mini-Fit_Jr_5566-04A_2x02_P4.20mm_Vertical
- J10: value Conn_01x03_Pin -> Conn_01x02_Pin; footprint Connector_Molex:Molex_KK-254_AE-6410-03A_1x03_P2.54mm_Vertical -> Minifit:Molex_Mini-Fit_Jr_5566-02A_2x01_P4.20mm_Vertical
- J11: footprint Connector_PinHeader_2.54mm:PinHeader_1x02_P2.54mm_Vertical -> Minifit:Molex_Mini-Fit_Jr_5566-02A_2x01_P4.20mm_Vertical
- J12, J18: value Conn_01x02_Pin -> Conn_02x07_Odd_Even; footprint Connector_PinHeader_2.54mm:PinHeader_1x02_P2.54mm_Vertical -> Connector_IDC:IDC-Header_2x07_P2.54mm_Latch_Vertical
- J13, J20: value Conn_02x07_Odd_Even -> Conn_01x02_Pin; footprint Connector_IDC:IDC-Header_2x07_P2.54mm_Latch_Vertical -> Connector_PinHeader_2.54mm:PinHeader_1x02_P2.54mm_Vertical
- J14: footprint Modules:Molex_Mini-Fit_Jr_5566-02A_2x01_P4.20mm_Vertical -> Connector_PinHeader_2.54mm:PinHeader_1x02_P2.54mm_Vertical
- J15: value Conn_01x02_Pin -> Conn_02x07_Odd_Even; footprint Modules:Molex_Mini-Fit_Jr_5566-02A_2x01_P4.20mm_Vertical -> Connector_IDC:IDC-Header_2x07_P2.54mm_Latch_Vertical
- J16: value Conn_01x03_Pin -> Conn_01x02_Pin; footprint Connector_Molex:Molex_KK-254_AE-6410-03A_1x03_P2.54mm_Vertical -> Connector_PinHeader_2.54mm:PinHeader_1x02_P2.54mm_Vertical
- J17: value Conn_02x02_ZigZag -> Conn_01x02_Pin; footprint Modules:Molex_Mini-Fit_Jr_5566-04A_2x02_P4.20mm_Vertical -> Connector_PinHeader_2.54mm:PinHeader_1x02_P2.54mm_Vertical
- J2: value Conn_01x02_Pin -> Conn_02x03; footprint Connector_Molex:Molex_KK-254_AE-6410-02A_1x02_P2.54mm_Vertical -> Minifit:Molex_Mini-Fit_Jr_5566-06A_2x03_P4.20mm_Vertical
- J3: value Conn_01x02_Pin -> Conn_02x02; footprint Connector_Molex:Molex_KK-254_AE-6410-02A_1x02_P2.54mm_Vertical -> Minifit:Molex_Mini-Fit_Jr_5566-04A_2x02_P4.20mm_Vertical
- J4: value Conn_02x02_ZigZag -> Conn_01x02_Pin; footprint Modules:Molex_Mini-Fit_Jr_5566-04A_2x02_P4.20mm_Vertical -> Connector_Molex:Molex_KK-254_AE-6410-02A_1x02_P2.54mm_Vertical
- J5: value Conn_01x03_Pin -> Conn_01x02_Pin; footprint Connector_Molex:Molex_KK-254_AE-6410-03A_1x03_P2.54mm_Vertical -> Connector_Molex:Molex_KK-254_AE-6410-02A_1x02_P2.54mm_Vertical
- J6, J8: value Conn_01x02_Pin -> Conn_01x03_Pin; footprint Connector_PinHeader_2.54mm:PinHeader_1x02_P2.54mm_Vertical -> Connector_Molex:Molex_KK-254_AE-6410-03A_1x03_P2.54mm_Vertical
- J9: value Conn_02x07_Odd_Even -> Conn_01x03_Pin; footprint Connector_IDC:IDC-Header_2x07_P2.54mm_Latch_Vertical -> Connector_Molex:Molex_KK-254_AE-6410-03A_1x03_P2.54mm_Vertical
- R10, R21, R34: value 47 -> 10k
- R12: value 91 -> 3k3
- R13: value 91 -> 10k
- R14, R15: value 150 -> 10k
- R16: value 1k5 -> 47
- R17, R31: value 1k5 -> 10k
- R19, R26, R33, R5: value 10k -> 3k3
- R2: value 4k7 -> 2k7
- R23: value 10k -> 47
- R24: value 3k3 -> 10k
- R27, R28, R29: value 1k -> 10k
- R3: value 2k7 -> 91
- R30: value 470 -> 47
- R32: value 1k2 -> 10k
- R35: value 3k3 -> 1k
- R36, R37, R38, R39: value 10k -> 1k
- R4: value 3k3 -> 4k7
- R41: value 1k -> ${R_in}
- R42: value 1k -> ${R_1}
- R43: value 150 -> ${R_2}
- R44: value 150 -> ${R_out_pullup}
- R45, R55: value 1k5 -> ${R_in}
- R46: value 1k2 -> ${R_in_bjt}
- R47: value 10k -> ${R_base_emitter}
- R48: value 47 -> ${R_pullup_bjt}
- R49: value 10k -> ${R_out_pullup}
- R50: value 10k -> ${R_in}
- R51: value 3k3 -> ${R_in_bjt}
- R52, R57: value 470 -> ${R_base_emitter}
- R53: value 150 -> ${R_pullup_bjt}
- R54: value 1k5 -> ${R_out_pullup}
- R56: value 150 -> ${R_in_bjt}
- R58: value 1k2 -> ${R_pullup_bjt}
- R6: value 10k -> 91
- R9: value 3k3 -> 47
- U1: value LV25-P -> LM324; footprint Sensor_Voltage:LEM_LV25-P -> Package_DIP:DIP-14_W7.62mm
- U10: value H11L1 -> ESP32-DevKitC; footprint Package_DIP:DIP-6_W7.62mm -> Espressif:ESP32-DevKitC
- U11: value H11L1 -> TL072; footprint Package_DIP:DIP-6_W7.62mm -> Package_DIP:DIP-8_W7.62mm
- U12: value LM324 -> HEF4093B
- U13: value HEF4093B -> TL072; footprint Package_DIP:DIP-14_W7.62mm -> Package_DIP:DIP-8_W7.62mm
- U14: value H11L1 -> HEF4093B; footprint Package_DIP:DIP-6_W7.62mm -> Package_DIP:DIP-14_W7.62mm
- U15: value LM324 -> TL072; footprint Package_DIP:DIP-14_W7.62mm -> Package_DIP:DIP-8_W7.62mm
- U16: value ESP32-DevKitC -> HEF4093B; footprint Espressif:ESP32-DevKitC -> Package_DIP:DIP-14_W7.62mm
- U18: value HEF4093B -> H11L1; footprint Package_DIP:DIP-14_W7.62mm -> Package_DIP:DIP-6_W7.62mm
- U21: value ~ -> H11L1; footprint Modules:TJA1050 -> Package_DIP:DIP-6_W7.62mm
- U3: value LM324 -> LV25-P; footprint Package_DIP:DIP-14_W7.62mm -> Sensor_Voltage:LEM_LV25-P
- U5, U7: value H11L1 -> LM324; footprint Package_DIP:DIP-6_W7.62mm -> Package_DIP:DIP-14_W7.62mm
- U6: value HEF4093B -> LM324
- U8: value LM324 -> ESP32-DevKitC; footprint Package_DIP:DIP-14_W7.62mm -> Espressif:ESP32-DevKitC
- U9: value ESP32-DevKitC -> TJA1050; footprint Espressif:ESP32-DevKitC -> CAN Modules:TJA1050
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Connections:
- C10 pad 1: +15V -> /V_read_in
- C10 pad 2: -15V -> GND
- C11 pad 1: /V_read_in -> /V_read_out
- C12 pad 1: /V_read_out -> /I_read_L1
- C13 pad 1: +3.3V -> /I_read_L2
- C14 pad 1: Vdrive -> /I_read_L3
- C14 pad 2: GND1 -> GND
- C15 pad 1: /PWM - 15V Level Shifter/Conectores - PWM e erro/erro_driver -> /I_read_out
- C15 pad 2: Net-(C34-Pad2) -> GND
- C16 pad 1: Vdrive -> +5V
- C16 pad 2: GND1 -> GND
- C17 pad 1: +15V -> +5V
- C17 pad 2: -15V -> GND
- C18 pad 1: /I_read_out -> +5V
- C19 pad 1: /I_read_L1 -> +5V
- C20 pad 1: /I_read_L3 -> +5V
- C21 pad 1: /I_read_L2 -> Net-(U11C-V+)
- C21 pad 2: GND -> Net-(U11C-V-)
- C22 pad 1: /PWM_TOP_2 -> Vdrive
- C22 pad 2: Net-(C15-Pad2) -> GND
- C23 pad 1: /PWM_BOT_2 -> Net-(U13C-V+)
- C23 pad 2: Net-(C17-Pad2) -> Net-(U13C-V-)
- C24 pad 2: GND1 -> GND
- C25 pad 1: /PWM - 15V Level Shifter/Conectores - PWM e erro1/erro_driver -> Net-(U15C-V+)
- C25 pad 2: Net-(C19-Pad2) -> Net-(U15C-V-)
- C26 pad 1: +15V -> Vdrive
- C26 pad 2: -15V -> GND
- C27 pad 1: +5V -> /Adequação Sinais Driver/Conectores - PWM e erro/erro_driver
- C27 pad 2: GND -> Net-(C27-Pad2)
- C28 pad 1: +5V -> +3.3V
- C29 pad 1: +5V -> /PWM_BOT_1
- C29 pad 2: GND -> Net-(C29-Pad2)
- C30 pad 1: +3.3V -> Vdrive
- C31 pad 1: /PWM_TOP_3 -> /PWM_TOP_1
- C31 pad 2: Net-(C22-Pad2) -> Net-(C31-Pad2)
- C32 pad 2: GND1 -> GND
- C33 pad 1: Vdrive -> /PWM_TOP_2
- C33 pad 2: GND1 -> Net-(C33-Pad2)
- C34 pad 2: GND1 -> GND
- C35 pad 1: +3.3V -> /PWM_TOP_3
- C35 pad 2: GND -> Net-(C35-Pad2)
- C36 pad 1: /PWM_BOT_3 -> Vdrive
- C36 pad 2: Net-(C24-Pad2) -> GND
- C37 pad 1: /PWM - 15V Level Shifter/Conectores - PWM e erro2/erro_driver -> /Adequação Sinais Driver/Conectores - PWM e erro1/erro_driver
- C37 pad 2: Net-(C26-Pad2) -> Net-(C37-Pad2)
- C5 pad 1: /PWM_TOP_1 -> +15V
- C5 pad 2: Net-(C36-Pad2) -> -15V
- C6 pad 1: /PWM_BOT_1 -> +15V
- C6 pad 2: Net-(C32-Pad2) -> -15V
- C7 pad 1: Vdrive -> +15V
- C7 pad 2: GND1 -> -15V
- C8 pad 1: Vdrive -> +15V
- C8 pad 2: GND1 -> -15V
- C9 pad 1: Vdrive -> +15V
- C9 pad 2: GND1 -> -15V
- F1 pad 1: /Power Connectors/+15V_sym_conn -> /Conectores/5V_conn
- F1 pad 2: +15V -> +5V
- F2 pad 1: /Power Connectors/-15V_sym_conn -> /Conectores/+15V_sym_conn
- F2 pad 2: -15V -> +15V
- F3 pad 1: /Power Connectors/Vdrive_conn -> /Conectores/-15V_sym_conn
- F3 pad 2: Vdrive -> -15V
- F4 pad 1: /Power Connectors/5V_conn -> /Conectores/Vdrive_conn
- F4 pad 2: +5V -> Vdrive
- J1 pad 1: /Power Connectors/-15V_sym_conn -> /Conectores/5V_conn
- J1 pad 3: /Power Connectors/+15V_sym_conn -> /Conectores/5V_conn
- J1 pad 4: /Power Connectors/-15V_sym_conn -> GND
- J10 pad 1: +15V -> /Microcontrolados e CAN/CANL
- J10 pad 2: Net-(J8-Pin_2) -> /Microcontrolados e CAN/CANH
- J11 pad 1: /PWM - 15V Level Shifter/Conectores - PWM e erro1/PWM_BOT_driver -> /Microcontrolados e CAN/CANL
- J11 pad 2: GND1 -> /Microcontrolados e CAN/CANH
- J12 pad 1: /PWM - 15V Level Shifter/Conectores - PWM e erro1/PWM_TOP_driver -> unconnected-(J12-Pin_1-Pad1)
- J12 pad 2: GND1 -> /Adequação Sinais Driver/Conectores - PWM e erro/PWM_BOT_driver
- J13 pad 1: unconnected-(J10-Pin_1-Pad1) -> /Adequação Sinais Driver/Conectores - PWM e erro/PWM_BOT_driver
- J13 pad 2: /PWM - 15V Level Shifter/Conectores - PWM e erro1/PWM_BOT_driver -> GND
- J14 pad 1: /MicroControladores/CANL -> /Adequação Sinais Driver/Conectores - PWM e erro/PWM_TOP_driver
- J14 pad 2: /MicroControladores/CANH -> GND
- J15 pad 1: /MicroControladores/CANL -> unconnected-(J15-Pin_1-Pad1)
- J15 pad 2: /MicroControladores/CANH -> /Adequação Sinais Driver/Conectores - PWM e erro1/PWM_BOT_driver
- J16 pad 1: +15V -> /Adequação Sinais Driver/Conectores - PWM e erro1/PWM_BOT_driver
- J16 pad 2: Net-(J9-Pin_2) -> GND
- J17 pad 1: /Power Connectors/5V_conn -> /Adequação Sinais Driver/Conectores - PWM e erro1/PWM_TOP_driver
- J18 pad 1: /PWM - 15V Level Shifter/Conectores - PWM e erro2/PWM_TOP_driver -> unconnected-(J18-Pin_1-Pad1)
- J18 pad 2: GND1 -> /Adequação Sinais Driver/Conectores - PWM e erro2/PWM_BOT_driver
- J19 pad 1: /PWM - 15V Level Shifter/Conectores - PWM e erro2/PWM_BOT_driver -> /Adequação Sinais Driver/Conectores - PWM e erro2/PWM_BOT_driver
- J19 pad 2: GND1 -> GND
- J2 pad 1: Net-(J2-Pin_1) -> /Conectores/-15V_sym_conn
- J2 pad 2: Net-(J2-Pin_2) -> GND
- J20 pad 1: unconnected-(J13-Pin_1-Pad1) -> /Adequação Sinais Driver/Conectores - PWM e erro2/PWM_TOP_driver
- J20 pad 2: /PWM - 15V Level Shifter/Conectores - PWM e erro2/PWM_BOT_driver -> GND
- J3 pad 1: Net-(J3-Pin_1) -> /Conectores/Vdrive_conn
- J3 pad 2: Net-(J3-Pin_2) -> GND
- J4 pad 1: /Power Connectors/Vdrive_conn -> Net-(J4-Pin_1)
- J4 pad 2: GND1 -> Net-(J4-Pin_2)
- J5 pad 1: +15V -> Net-(J5-Pin_1)
- J5 pad 2: Net-(J1-Pin_2) -> Net-(J5-Pin_2)
- J6 pad 1: /PWM - 15V Level Shifter/Conectores - PWM e erro/PWM_TOP_driver -> +15V
- J6 pad 2: GND1 -> Net-(J6-Pin_2)
- J8 pad 1: /PWM - 15V Level Shifter/Conectores - PWM e erro/PWM_BOT_driver -> +15V
- J8 pad 2: GND1 -> Net-(J8-Pin_2)
- J9 pad 1: unconnected-(J16-Pin_1-Pad1) -> +15V
- J9 pad 2: /PWM - 15V Level Shifter/Conectores - PWM e erro/PWM_BOT_driver -> Net-(J9-Pin_2)
- J9 pad 3: /PWM - 15V Level Shifter/Conectores - PWM e erro/erro_driver -> -15V
- R1 pad 1: Net-(R8-Pad2) -> Net-(J4-Pin_1)
- R1 pad 2: Net-(U2-HV+) -> Net-(R1-Pad2)
- R10 pad 1: GND -> Net-(U4B-+)
- R10 pad 2: Net-(J1-Pin_2) -> Net-(U4A--)
- R11 pad 1: +3.3V -> Net-(U4B-+)
- R11 pad 2: Net-(U1C-+) -> Net-(U4C--)
- R12 pad 1: GND -> Net-(U4B--)
- R12 pad 2: /Adequação Sinais Corrente e Tensão/adequacao_sensor_tensao1/output_signal -> GND
- R13 pad 1: GND -> /Adequação Sensores/Filtro RC2/unfilt_signal
- R13 pad 2: /Adequação Sinais Corrente e Tensão/adequacao_sensor_tensao/output_signal -> Net-(U4B-+)
- R14 pad 1: /PWM_BOT_1 -> +3.3V
- R14 pad 2: Net-(C32-Pad2) -> Net-(U5C-+)
- R15 pad 1: /PWM_TOP_1 -> Net-(U5C-+)
- R15 pad 2: Net-(C36-Pad2) -> GND
- R16 pad 1: Vdrive -> GND
- R16 pad 2: /PWM - 15V Level Shifter/Conectores - PWM e erro/Isolação de sinais - PWM7/output_sign -> Net-(J7-Pin_2)
- R17 pad 1: Vdrive -> Net-(U5B-+)
- R17 pad 2: /PWM - 15V Level Shifter/Conectores - PWM e erro/Isolação de sinais - PWM6/output_sign -> Net-(U5A--)
- R18 pad 2: Net-(U5A--) -> Net-(U5C--)
- R19 pad 1: Net-(U5C-+) -> Net-(U5B--)
- R2 pad 1: Net-(J2-Pin_1) -> Net-(R1-Pad2)
- R2 pad 2: Net-(R8-Pad2) -> Net-(U2-HV+)
- R20 pad 1: Net-(U5B-+) -> /Adequação Sensores/Filtro RC3/unfilt_signal
- R20 pad 2: Net-(U5C--) -> Net-(U5B-+)
- R21 pad 1: GND -> +3.3V
- R21 pad 2: Net-(J7-Pin_2) -> Net-(U6C-+)
- R23 pad 1: +3.3V -> GND
- R23 pad 2: Net-(U5C-+) -> Net-(J8-Pin_2)
- R24 pad 1: Net-(U5B--) -> Net-(U6B-+)
- R24 pad 2: GND -> Net-(U6A--)
- R25 pad 1: +3.3V -> Net-(U6B-+)
- R25 pad 2: Net-(U6C-+) -> Net-(U6C--)
- R26 pad 1: /Adequação Sinais Corrente e Tensão/Filtro RC3/unfilt_signal -> Net-(U6B--)
- R26 pad 2: Net-(U5B-+) -> GND
- R27 pad 1: /Adequação Sinais Corrente e Tensão/Filtro RC1/unfilt_signal -> /Adequação Sensores/Filtro RC4/unfilt_signal
- R27 pad 2: /V_read_out -> Net-(U6B-+)
- R28 pad 1: /Adequação Sinais Corrente e Tensão/Filtro RC2/unfilt_signal -> +3.3V
- R28 pad 2: /I_read_L1 -> Net-(U7C-+)
- R29 pad 1: /Adequação Sinais Corrente e Tensão/Filtro RC/unfilt_signal -> Net-(U7C-+)
- R29 pad 2: /V_read_in -> GND
- R3 pad 1: Net-(R11-Pad2) -> GND
- R3 pad 2: Net-(U3-HV+) -> /Adequação Sensores/adequacao_sensor_tensao/output_signal
- R30 pad 1: +3.3V -> GND
- R30 pad 2: /err_1 -> Net-(J9-Pin_2)
- R31 pad 1: Vdrive -> Net-(U7B-+)
- R31 pad 2: /PWM - 15V Level Shifter/Conectores - PWM e erro1/Isolação de sinais - PWM7/output_sign -> Net-(U7A--)
- R32 pad 1: /PWM - 15V Level Shifter/Conectores - PWM e erro/erro_driver -> Net-(U7B-+)
- R32 pad 2: Net-(C34-Pad2) -> Net-(U7C--)
- R33 pad 1: +3.3V -> Net-(U7B--)
- R33 pad 2: Net-(U7C-+) -> GND
- R34 pad 1: GND -> /Adequação Sensores/Filtro RC5/unfilt_signal
- R34 pad 2: Net-(J8-Pin_2) -> Net-(U7B-+)
- R35 pad 1: Net-(U6B--) -> /Adequação Sensores/Filtro RC/unfilt_signal
- R35 pad 2: GND -> /V_read_in
- R36 pad 1: Net-(U6B-+) -> /Adequação Sensores/Filtro RC1/unfilt_signal
- R36 pad 2: Net-(U6C--) -> /V_read_out
- R37 pad 1: Net-(U6B-+) -> /Adequação Sensores/Filtro RC2/unfilt_signal
- R37 pad 2: Net-(U6A--) -> /I_read_L1
- R38 pad 1: Net-(U7C-+) -> /Adequação Sensores/Filtro RC3/unfilt_signal
- R38 pad 2: GND -> /I_read_L2
- R39 pad 1: /Adequação Sinais Corrente e Tensão/Filtro RC4/unfilt_signal -> /Adequação Sensores/Filtro RC4/unfilt_signal
- R39 pad 2: Net-(U6B-+) -> /I_read_L3
- R4 pad 1: Net-(J3-Pin_1) -> Net-(J5-Pin_1)
- R4 pad 2: Net-(R11-Pad2) -> Net-(R4-Pad2)
- R40 pad 1: /Adequação Sinais Corrente e Tensão/Filtro RC5/unfilt_signal -> /Adequação Sensores/Filtro RC5/unfilt_signal
- R41 pad 1: /Adequação Sinais Corrente e Tensão/Filtro RC4/unfilt_signal -> /Adequação Sinais Driver/Conectores - PWM e erro/erro_driver
- R41 pad 2: /I_read_L3 -> Net-(C27-Pad2)
- R42 pad 1: /Adequação Sinais Corrente e Tensão/Filtro RC3/unfilt_signal -> Net-(R42-Pad1)
- R42 pad 2: /I_read_L2 -> /Adequação Sinais Driver/Conectores - PWM e erro/erro_driver
- R43 pad 1: /PWM_BOT_2 -> GND
- R43 pad 2: Net-(C17-Pad2) -> Net-(R42-Pad1)
- R44 pad 1: /PWM_TOP_2 -> +3.3V
- R44 pad 2: Net-(C15-Pad2) -> /err_1
- R45 pad 1: Vdrive -> /PWM_BOT_1
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Routing:
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- removed copper zone on B.Cu, net GND
- removed copper zone on F.Cu, net GND
- removed copper zone on B.Cu, net GND1
- removed copper zone on F.Cu, net GND1
Other:
- board outline removed
- board text removed: "15V"
- board text removed: "5V"
- board text removed: "BOT"
- board text removed: "CANH"
- board text removed: "CANL"
- board text removed: "TOP"
- board text removed: "± 15V"

Commit message: Modificações nas duas placas, adição de furos para montagem, melhora na posição dos micros e conectores para comunicação SPI
Parts:
- removed C40, C42, C44: 0,1u, Capacitor_THT:C_Disc_D8.0mm_W5.0mm_P7.50mm
- removed C41, C43: ${C_in}, Capacitor_THT:C_Disc_D8.0mm_W5.0mm_P7.50mm
- removed R52, R57, R71, R80: ${R_base_emitter}, Resistor_THT:R_Axial_DIN0207_L6.3mm_D2.5mm_P7.62mm_Horizontal
- removed R55, R60, R69, R74: ${R_in}, Resistor_THT:R_Axial_DIN0207_L6.3mm_D2.5mm_P7.62mm_Horizontal
- removed R66: ${R_1}, Resistor_THT:R_Axial_DIN0207_L6.3mm_D2.5mm_P7.62mm_Horizontal
- removed RV1, RV2, RV3, RV4: Varistor, Varistor:RV_Disc_D12mm_W3.9mm_P7.5mm
- added G***: LOGO, Logos:logo_poli_13mm, F.Cu at (106.1, 79.9)
- added H1: MountingHole_Pad, MountingHole:MountingHole_3.2mm_M3_Pad_Via, F.Cu at (170.0, 80.3)
- added H2: MountingHole_Pad, MountingHole:MountingHole_3.2mm_M3_Pad_Via, F.Cu at (39.6, 144.4)
- added H3: MountingHole_Pad, MountingHole:MountingHole_3.2mm_M3_Pad_Via, F.Cu at (38.7, 60.0)
- added J21: Conn_01x04_Pin, Connector_Molex:Molex_KK-254_AE-6410-04A_1x04_P2.54mm_Vertical, F.Cu at (52.8, 81.2)
- added J22: Conn_01x04_Pin, Connector_Molex:Molex_KK-254_AE-6410-04A_1x04_P2.54mm_Vertical, F.Cu at (153.3, 118.3)
- added R84: 1k, Resistor_SMD:R_0805_2012Metric_Pad1.20x1.40mm_HandSolder, F.Cu at (49.8, 54.7)
- added R86: 180, Resistor_SMD:R_0805_2012Metric_Pad1.20x1.40mm_HandSolder, F.Cu at (61.9, 71.0)
- added R87: 100k, Resistor_SMD:R_0805_2012Metric_Pad1.20x1.40mm_HandSolder, F.Cu at (61.7, 63.5)
- added R89: 1k, Resistor_SMD:R_0805_2012Metric_Pad1.20x1.40mm_HandSolder, F.Cu at (61.9, 54.7)
- C10, C11, C12, C13, C2, C21, C23, C24, C25, C26, C28, C30, C4, C6, C7: footprint Capacitor_THT:C_Disc_D8.0mm_W5.0mm_P7.50mm -> Capacitor_SMD:C_0805_2012Metric_Pad1.18x1.45mm_HandSolder
- C14, C15: value 330n -> 0,1u; footprint Capacitor_THT:C_Disc_D8.0mm_W5.0mm_P7.50mm -> Capacitor_SMD:C_0805_2012Metric_Pad1.18x1.45mm_HandSolder
- C18: value 10u -> 0,1u; footprint Capacitor_SMD:C_1210_3225Metric_Pad1.33x2.70mm_HandSolder -> Capacitor_SMD:C_0805_2012Metric_Pad1.18x1.45mm_HandSolder
- C20: value 10u -> 6,8n; footprint Capacitor_SMD:C_1210_3225Metric_Pad1.33x2.70mm_HandSolder -> Capacitor_SMD:C_0805_2012Metric_Pad1.18x1.45mm_HandSolder
- C22, C36, C38: value 0,1u -> 6,8n; footprint Capacitor_THT:C_Disc_D8.0mm_W5.0mm_P7.50mm -> Capacitor_SMD:C_0805_2012Metric_Pad1.18x1.45mm_HandSolder
- C27, C29: value ${C_in} -> 6,8n; footprint Capacitor_THT:C_Disc_D8.0mm_W5.0mm_P7.50mm -> Capacitor_SMD:C_0805_2012Metric_Pad1.18x1.45mm_HandSolder
- C3, C5: value 4,7u -> 0,1u; footprint Capacitor_THT:C_Disc_D8.0mm_W5.0mm_P7.50mm -> Capacitor_SMD:C_0805_2012Metric_Pad1.18x1.45mm_HandSolder
- C31, C33, C35, C37, C39: value ${C_in} -> 0,1u; footprint Capacitor_THT:C_Disc_D8.0mm_W5.0mm_P7.50mm -> Capacitor_SMD:C_0805_2012Metric_Pad1.18x1.45mm_HandSolder
- C32, C34: value 0,1u -> 10u; footprint Capacitor_THT:C_Disc_D8.0mm_W5.0mm_P7.50mm -> Capacitor_SMD:C_1210_3225Metric_Pad1.33x2.70mm_HandSolder
- C8, C9: value 0,1u -> 330n; footprint Capacitor_THT:C_Disc_D8.0mm_W5.0mm_P7.50mm -> Capacitor_SMD:C_0805_2012Metric_Pad1.18x1.45mm_HandSolder
- F1, F2, F3, F4: footprint Fuse:Fuse_BelFuse_0ZRE0005FF_L8.3mm_W3.8mm -> Fuse:Fuse_1210_3225Metric_Pad1.42x2.65mm_HandSolder
- J12, J15, J18: footprint Connector_IDC:IDC-Header_2x07_P2.54mm_Latch_Vertical -> IDC Connectors:IDC_Header_2x07
- R1: value 3k3 -> 3k3 1W; footprint Resistor_THT:R_Axial_DIN0207_L6.3mm_D2.5mm_P7.62mm_Horizontal -> Resistor_THT:R_Axial_DIN0614_L14.3mm_D5.7mm_P5.08mm_Vertical
- R10, R17, R18, R25, R34: value 10k -> 91 1/8W; footprint Resistor_THT:R_Axial_DIN0207_L6.3mm_D2.5mm_P7.62mm_Horizontal -> Resistor_SMD:R_0805_2012Metric_Pad1.20x1.40mm_HandSolder
- R11, R14, R15, R20, R22, R24, R27, R28, R31, R32, R39, R40, R7, R8: footprint Resistor_THT:R_Axial_DIN0207_L6.3mm_D2.5mm_P7.62mm_Horizontal -> Resistor_SMD:R_0805_2012Metric_Pad1.20x1.40mm_HandSolder
- R12, R19: value 3k3 -> 10k; footprint Resistor_THT:R_Axial_DIN0207_L6.3mm_D2.5mm_P7.62mm_Horizontal -> Resistor_SMD:R_0805_2012Metric_Pad1.20x1.40mm_HandSolder
- R13, R21, R29: value 10k -> 3k3; footprint Resistor_THT:R_Axial_DIN0207_L6.3mm_D2.5mm_P7.62mm_Horizontal -> Resistor_SMD:R_0805_2012Metric_Pad1.20x1.40mm_HandSolder
- R16, R23, R30: value 47 -> 10k; footprint Resistor_THT:R_Axial_DIN0207_L6.3mm_D2.5mm_P7.62mm_Horizontal -> Resistor_SMD:R_0805_2012Metric_Pad1.20x1.40mm_HandSolder
- R2: value 2k7 -> 2k7 1W; footprint Resistor_THT:R_Axial_DIN0207_L6.3mm_D2.5mm_P7.62mm_Horizontal -> Resistor_THT:R_Axial_DIN0516_L15.5mm_D5.0mm_P5.08mm_Vertical
- R26, R33: value 3k3 -> 91 1/8W; footprint Resistor_THT:R_Axial_DIN0207_L6.3mm_D2.5mm_P7.62mm_Horizontal -> Resistor_SMD:R_0805_2012Metric_Pad1.20x1.40mm_HandSolder
- R3, R6: value 91 -> 91 1/8W; footprint Resistor_THT:R_Axial_DIN0207_L6.3mm_D2.5mm_P7.62mm_Horizontal -> Resistor_SMD:R_0805_2012Metric_Pad1.20x1.40mm_HandSolder
- R35, R36, R38: value 1k -> 10k; footprint Resistor_THT:R_Axial_DIN0207_L6.3mm_D2.5mm_P7.62mm_Horizontal -> Resistor_SMD:R_0805_2012Metric_Pad1.20x1.40mm_HandSolder
- R37: value 1k -> 3k3; footprint Resistor_THT:R_Axial_DIN0207_L6.3mm_D2.5mm_P7.62mm_Horizontal -> Resistor_SMD:R_0805_2012Metric_Pad1.20x1.40mm_HandSolder
- R4: value 4k7 -> 4k7 2W; footprint Resistor_THT:R_Axial_DIN0207_L6.3mm_D2.5mm_P7.62mm_Horizontal -> Resistor_THT:R_Axial_DIN0614_L14.3mm_D5.7mm_P5.08mm_Vertical
- R41, R65: value ${R_in} -> 1k; footprint Resistor_THT:R_Axial_DIN0207_L6.3mm_D2.5mm_P7.62mm_Horizontal -> Resistor_SMD:R_0805_2012Metric_Pad1.20x1.40mm_HandSolder
- R42, R75: value ${R_1} -> 1k; footprint Resistor_THT:R_Axial_DIN0207_L6.3mm_D2.5mm_P7.62mm_Horizontal -> Resistor_SMD:R_0805_2012Metric_Pad1.20x1.40mm_HandSolder
- R43: value ${R_2} -> 1k; footprint Resistor_THT:R_Axial_DIN0207_L6.3mm_D2.5mm_P7.62mm_Horizontal -> Resistor_SMD:R_0805_2012Metric_Pad1.20x1.40mm_HandSolder
- R44: value ${R_out_pullup} -> 1k; footprint Resistor_THT:R_Axial_DIN0207_L6.3mm_D2.5mm_P7.62mm_Horizontal -> Resistor_SMD:R_0805_2012Metric_Pad1.20x1.40mm_HandSolder
- R45: value ${R_in} -> 100; footprint Resistor_THT:R_Axial_DIN0207_L6.3mm_D2.5mm_P7.62mm_Horizontal -> Resistor_SMD:R_0805_2012Metric_Pad1.20x1.40mm_HandSolder
- R46: value ${R_in_bjt} -> 10k; footprint Resistor_THT:R_Axial_DIN0207_L6.3mm_D2.5mm_P7.62mm_Horizontal -> Resistor_SMD:R_0805_2012Metric_Pad1.20x1.40mm_HandSolder
- R47: value ${R_base_emitter} -> 20k; footprint Resistor_THT:R_Axial_DIN0207_L6.3mm_D2.5mm_P7.62mm_Horizontal -> Resistor_SMD:R_0805_2012Metric_Pad1.20x1.40mm_HandSolder
- R48: value ${R_pullup_bjt} -> 1k3; footprint Resistor_THT:R_Axial_DIN0207_L6.3mm_D2.5mm_P7.62mm_Horizontal -> Resistor_SMD:R_0805_2012Metric_Pad1.20x1.40mm_HandSolder
- R49, R77: value ${R_out_pullup} -> 39k; footprint Resistor_THT:R_Axial_DIN0207_L6.3mm_D2.5mm_P7.62mm_Horizontal -> Resistor_SMD:R_0805_2012Metric_Pad1.20x1.40mm_HandSolder
- R5: value 3k3 -> 3k3 1/2W; footprint Resistor_THT:R_Axial_DIN0207_L6.3mm_D2.5mm_P7.62mm_Horizontal -> Resistor_THT:R_Axial_DIN0516_L15.5mm_D5.0mm_P5.08mm_Vertical
- R50, R78: value ${R_in} -> 11k; footprint Resistor_THT:R_Axial_DIN0207_L6.3mm_D2.5mm_P7.62mm_Horizontal -> Resistor_SMD:R_0805_2012Metric_Pad1.20x1.40mm_HandSolder
- R51, R56, R61, R70, R79: value ${R_in_bjt} -> 1k; footprint Resistor_THT:R_Axial_DIN0207_L6.3mm_D2.5mm_P7.62mm_Horizontal -> Resistor_SMD:R_0805_2012Metric_Pad1.20x1.40mm_HandSolder
- R53, R58, R72, R81: value ${R_pullup_bjt} -> 180; footprint Resistor_THT:R_Axial_DIN0207_L6.3mm_D2.5mm_P7.62mm_Horizontal -> Resistor_SMD:R_0805_2012Metric_Pad1.20x1.40mm_HandSolder
- R54, R59, R68, R73, R82: value ${R_out_pullup} -> 100k; footprint Resistor_THT:R_Axial_DIN0207_L6.3mm_D2.5mm_P7.62mm_Horizontal -> Resistor_SMD:R_0805_2012Metric_Pad1.20x1.40mm_HandSolder
- R62: value ${R_base_emitter} -> 1k3; footprint Resistor_THT:R_Axial_DIN0207_L6.3mm_D2.5mm_P7.62mm_Horizontal -> Resistor_SMD:R_0805_2012Metric_Pad1.20x1.40mm_HandSolder
- R63: value ${R_pullup_bjt} -> 39k; footprint Resistor_THT:R_Axial_DIN0207_L6.3mm_D2.5mm_P7.62mm_Horizontal -> Resistor_SMD:R_0805_2012Metric_Pad1.20x1.40mm_HandSolder
- R64: value ${R_out_pullup} -> 11k; footprint Resistor_THT:R_Axial_DIN0207_L6.3mm_D2.5mm_P7.62mm_Horizontal -> Resistor_SMD:R_0805_2012Metric_Pad1.20x1.40mm_HandSolder
- R67: value ${R_2} -> 180; footprint Resistor_THT:R_Axial_DIN0207_L6.3mm_D2.5mm_P7.62mm_Horizontal -> Resistor_SMD:R_0805_2012Metric_Pad1.20x1.40mm_HandSolder
- R76: value ${R_2} -> 1k3; footprint Resistor_THT:R_Axial_DIN0207_L6.3mm_D2.5mm_P7.62mm_Horizontal -> Resistor_SMD:R_0805_2012Metric_Pad1.20x1.40mm_HandSolder
- R9: value 47 -> 91 1/8W; footprint Resistor_THT:R_Axial_DIN0207_L6.3mm_D2.5mm_P7.62mm_Horizontal -> Resistor_SMD:R_0805_2012Metric_Pad1.20x1.40mm_HandSolder
- U1: value LM324 -> LM358; footprint Package_DIP:DIP-14_W7.62mm -> Package_DIP:DIP-8_W7.62mm
- U10: value ESP32-DevKitC -> HEF4093B; footprint Espressif:ESP32-DevKitC -> Package_DIP:DIP-14_W7.62mm
- U13, U15: value TL072 -> H11L1; footprint Package_DIP:DIP-8_W7.62mm -> Package_DIP:DIP-6_W7.62mm
- U14: value HEF4093B -> H11L1; footprint Package_DIP:DIP-14_W7.62mm -> Package_DIP:DIP-6_W7.62mm
- U16: value HEF4093B -> TL072; footprint Package_DIP:DIP-14_W7.62mm -> Package_DIP:DIP-8_W7.62mm
- U17: value H11L1 -> HEF4093B; footprint Package_DIP:DIP-6_W7.62mm -> Package_DIP:DIP-14_W7.62mm
- U21, U22: value H11L1 -> ESP32-DevKitC; footprint Package_DIP:DIP-6_W7.62mm -> Espressif:ESP32-DevKitC
- U8: value ESP32-DevKitC -> TJA1050; footprint Espressif:ESP32-DevKitC -> CAN Modules:TJA1050
- U9: value TJA1050 -> TL072; footprint CAN Modules:TJA1050 -> Package_DIP:DIP-8_W7.62mm
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Connections:
- C10 pad 1: /V_read_in -> /I_read_L1
- C11 pad 1: /V_read_out -> /I_read_L2
- C12 pad 1: /I_read_L1 -> /I_read_L3
- C13 pad 1: /I_read_L2 -> /I_read_out
- C14 pad 1: /I_read_L3 -> +5V
- C15 pad 1: /I_read_out -> Vdrive
- C16 pad 1: +5V -> Vdrive
- C17 pad 1: +5V -> Vdrive
- C18 pad 1: +5V -> Vdrive
- C19 pad 1: +5V -> +3.3V
- C20 pad 1: +5V -> /PWM_TOP_2
- C20 pad 2: GND -> /Adequação Sinais Driver/Conectores - PWM e erro1/Adequação Sinais - PWM1/in_sign_aux
- C21 pad 1: Net-(U11C-V+) -> Vdrive
- C21 pad 2: Net-(U11C-V-) -> GND
- C22 pad 1: Vdrive -> /PWM_BOT_2
- C22 pad 2: GND -> /Adequação Sinais Driver/Conectores - PWM e erro1/Adequação Sinais - PWM/in_sign_aux
- C23 pad 1: Net-(U13C-V+) -> Vdrive
- C23 pad 2: Net-(U13C-V-) -> GND
- C25 pad 1: Net-(U15C-V+) -> Vdrive
- C25 pad 2: Net-(U15C-V-) -> GND
- C26 pad 1: Vdrive -> +3.3V
- C27 pad 1: /Adequação Sinais Driver/Conectores - PWM e erro/erro_driver -> /PWM_TOP_3
- C27 pad 2: Net-(C27-Pad2) -> /Adequação Sinais Driver/Conectores - PWM e erro2/Adequação Sinais - PWM1/in_sign_aux
- C28 pad 1: +3.3V -> Vdrive
- C29 pad 1: /PWM_BOT_1 -> /PWM_BOT_3
- C29 pad 2: Net-(C29-Pad2) -> /Adequação Sinais Driver/Conectores - PWM e erro2/Adequação Sinais - PWM/in_sign_aux
- C31 pad 1: /PWM_TOP_1 -> +5V
- C31 pad 2: Net-(C31-Pad2) -> GND
- C32 pad 1: Vdrive -> +5V
- C33 pad 1: /PWM_TOP_2 -> +5V
- C33 pad 2: Net-(C33-Pad2) -> GND
- C34 pad 1: Vdrive -> +5V
- C35 pad 1: /PWM_TOP_3 -> +3.3V
- C35 pad 2: Net-(C35-Pad2) -> GND
- C36 pad 1: Vdrive -> /PWM_BOT_1
- C36 pad 2: GND -> /Adequação Sinais Driver/Conectores - PWM e erro/Adequação Sinais - PWM/in_sign_aux
- C37 pad 1: /Adequação Sinais Driver/Conectores - PWM e erro1/erro_driver -> Vdrive
- C37 pad 2: Net-(C37-Pad2) -> GND
- C38 pad 1: +3.3V -> /PWM_TOP_1
- C38 pad 2: GND -> /Adequação Sinais Driver/Conectores - PWM e erro/Adequação Sinais - PWM1/in_sign_aux
- C39 pad 1: /PWM_BOT_2 -> Vdrive
- C39 pad 2: Net-(C39-Pad2) -> GND
- C8 pad 1: +15V -> /V_read_in
- C8 pad 2: -15V -> GND
- C9 pad 1: +15V -> /V_read_out
- C9 pad 2: -15V -> GND
- Q1 pad 1: /Adequação Sinais Driver/Conectores - PWM e erro/PWM_TOP_int -> /Adequação Sinais Driver/Conectores - PWM e erro1/PWM_BOT_int
- Q1 pad 2: Net-(Q1-B) -> /Adequação Sinais Driver/Conectores - PWM e erro1/Adequação Sinais - PWM1/in_sign_aux
- Q2 pad 1: /Adequação Sinais Driver/Conectores - PWM e erro/PWM_BOT_int -> /Adequação Sinais Driver/Conectores - PWM e erro1/PWM_TOP_int
- Q2 pad 2: Net-(Q2-B) -> /Adequação Sinais Driver/Conectores - PWM e erro1/Adequação Sinais - PWM/in_sign_aux
- Q3 pad 1: /Adequação Sinais Driver/Conectores - PWM e erro1/PWM_BOT_int -> /Adequação Sinais Driver/Conectores - PWM e erro2/PWM_BOT_int
- Q3 pad 2: Net-(Q3-B) -> /Adequação Sinais Driver/Conectores - PWM e erro2/Adequação Sinais - PWM1/in_sign_aux
- Q4 pad 1: /Adequação Sinais Driver/Conectores - PWM e erro2/PWM_BOT_int -> /Adequação Sinais Driver/Conectores - PWM e erro2/PWM_TOP_int
- Q4 pad 2: Net-(Q4-B) -> /Adequação Sinais Driver/Conectores - PWM e erro2/Adequação Sinais - PWM/in_sign_aux
- Q5 pad 1: /Adequação Sinais Driver/Conectores - PWM e erro1/PWM_TOP_int -> /Adequação Sinais Driver/Conectores - PWM e erro/PWM_TOP_int
- Q5 pad 2: Net-(Q5-B) -> /Adequação Sinais Driver/Conectores - PWM e erro/Adequação Sinais - PWM/in_sign_aux
- Q6 pad 1: /Adequação Sinais Driver/Conectores - PWM e erro2/PWM_TOP_int -> /Adequação Sinais Driver/Conectores - PWM e erro/PWM_BOT_int
- Q6 pad 2: Net-(Q6-B) -> /Adequação Sinais Driver/Conectores - PWM e erro/Adequação Sinais - PWM1/in_sign_aux
- R10 pad 1: Net-(U4B-+) -> GND
- R10 pad 2: Net-(U4A--) -> Net-(J6-Pin_2)
- R11 pad 2: Net-(U4C--) -> Net-(U4A--)
- R12 pad 1: Net-(U4B--) -> Net-(U4B-+)
- R12 pad 2: GND -> Net-(U4C--)
- R13 pad 1: /Adequação Sensores/Filtro RC2/unfilt_signal -> Net-(U4B--)
- R13 pad 2: Net-(U4B-+) -> GND
- R14 pad 1: +3.3V -> /Adequação Sensores/Filtro RC2/unfilt_signal
- R14 pad 2: Net-(U5C-+) -> Net-(U4B-+)
- R15 pad 1: Net-(U5C-+) -> +3.3V
- R15 pad 2: GND -> Net-(U5C-+)
- R16 pad 1: GND -> Net-(U5C-+)
- R16 pad 2: Net-(J7-Pin_2) -> GND
- R17 pad 1: Net-(U5B-+) -> GND
- R17 pad 2: Net-(U5A--) -> Net-(J7-Pin_2)
- R18 pad 1: Net-(U5B-+) -> GND
- R18 pad 2: Net-(U5C--) -> Net-(J7-Pin_2)
- R19 pad 1: Net-(U5B--) -> Net-(U5B-+)
- R19 pad 2: GND -> Net-(U5A--)
- R2 pad 1: Net-(R1-Pad2) -> Net-(U2-HV+)
- R2 pad 2: Net-(U2-HV+) -> Net-(R1-Pad2)
- R20 pad 1: /Adequação Sensores/Filtro RC3/unfilt_signal -> Net-(U5B-+)
- R20 pad 2: Net-(U5B-+) -> Net-(U5C--)
- R21 pad 1: +3.3V -> Net-(U5B--)
- R21 pad 2: Net-(U6C-+) -> GND
- R22 pad 1: Net-(U6C-+) -> /Adequação Sensores/Filtro RC3/unfilt_signal
- R22 pad 2: GND -> Net-(U5B-+)
- R23 pad 1: GND -> +3.3V
- R23 pad 2: Net-(J8-Pin_2) -> Net-(U6C-+)
- R24 pad 1: Net-(U6B-+) -> Net-(U6C-+)
- R24 pad 2: Net-(U6A--) -> GND
- R25 pad 1: Net-(U6B-+) -> GND
- R25 pad 2: Net-(U6C--) -> Net-(J8-Pin_2)
- R26 pad 1: Net-(U6B--) -> GND
- R26 pad 2: GND -> Net-(J8-Pin_2)
- R27 pad 1: /Adequação Sensores/Filtro RC4/unfilt_signal -> Net-(U6B-+)
- R27 pad 2: Net-(U6B-+) -> Net-(U6A--)
- R28 pad 1: +3.3V -> Net-(U6B-+)
- R28 pad 2: Net-(U7C-+) -> Net-(U6C--)
- R29 pad 1: Net-(U7C-+) -> Net-(U6B--)
- R30 pad 1: GND -> /Adequação Sensores/Filtro RC4/unfilt_signal
- R30 pad 2: Net-(J9-Pin_2) -> Net-(U6B-+)
- R31 pad 1: Net-(U7B-+) -> +3.3V
- R31 pad 2: Net-(U7A--) -> Net-(U7C-+)
- R32 pad 1: Net-(U7B-+) -> Net-(U7C-+)
- R32 pad 2: Net-(U7C--) -> GND
- R33 pad 1: Net-(U7B--) -> GND
- R33 pad 2: GND -> Net-(J9-Pin_2)
- R34 pad 1: /Adequação Sensores/Filtro RC5/unfilt_signal -> GND
- R34 pad 2: Net-(U7B-+) -> Net-(J9-Pin_2)
- R35 pad 1: /Adequação Sensores/Filtro RC/unfilt_signal -> Net-(U7B-+)
- R35 pad 2: /V_read_in -> Net-(U7A--)
- R36 pad 1: /Adequação Sensores/Filtro RC1/unfilt_signal -> Net-(U7B-+)
- R36 pad 2: /V_read_out -> Net-(U7C--)
- R37 pad 1: /Adequação Sensores/Filtro RC2/unfilt_signal -> Net-(U7B--)
- R37 pad 2: /I_read_L1 -> GND
- R38 pad 1: /Adequação Sensores/Filtro RC3/unfilt_signal -> /Adequação Sensores/Filtro RC5/unfilt_signal
- R38 pad 2: /I_read_L2 -> Net-(U7B-+)
- R39 pad 1: /Adequação Sensores/Filtro RC4/unfilt_signal -> /Adequação Sensores/Filtro RC/unfilt_signal
- R39 pad 2: /I_read_L3 -> /V_read_in
- R40 pad 1: /Adequação Sensores/Filtro RC5/unfilt_signal -> /Adequação Sensores/Filtro RC1/unfilt_signal
- R40 pad 2: /I_read_out -> /V_read_out
- R41 pad 1: /Adequação Sinais Driver/Conectores - PWM e erro/erro_driver -> /Adequação Sensores/Filtro RC2/unfilt_signal
- R41 pad 2: Net-(C27-Pad2) -> /I_read_L1
- R42 pad 1: Net-(R42-Pad1) -> /Adequação Sensores/Filtro RC3/unfilt_signal
- R42 pad 2: /Adequação Sinais Driver/Conectores - PWM e erro/erro_driver -> /I_read_L2
- R43 pad 1: GND -> /Adequação Sensores/Filtro RC4/unfilt_signal
- R43 pad 2: Net-(R42-Pad1) -> /I_read_L3
- R44 pad 1: +3.3V -> /Adequação Sensores/Filtro RC5/unfilt_signal
- R44 pad 2: /err_1 -> /I_read_out
- R45 pad 1: /PWM_BOT_1 -> /Microcontrolados e CAN/CAN_TX_trans
- R45 pad 2: Net-(C29-Pad2) -> /Microcontrolados e CAN/CAN_TX_esp
- R46 pad 1: /PWM_BOT_1 -> /Microcontrolados e CAN/CAN_RX_trans
- R46 pad 2: Net-(Q1-B) -> /Microcontrolados e CAN/CAN_RX_esp
- R47 pad 1: Net-(Q1-B) -> /Microcontrolados e CAN/CAN_RX_esp
- R48 pad 1: Vdrive -> /Adequação Sinais Driver/Conectores - PWM e erro1/erro_driver
- R48 pad 2: /Adequação Sinais Driver/Conectores - PWM e erro/PWM_TOP_int -> Net-(R48-Pad2)
- R49 pad 1: Vdrive -> /err_2
- R49 pad 2: /Adequação Sinais Driver/Conectores - PWM e erro/PWM_TOP_int -> /Adequação Sinais Driver/Conectores - PWM e erro1/erro_driver
- R5 pad 1: Net-(R4-Pad2) -> Net-(U3-HV+)
- R5 pad 2: Net-(U3-HV+) -> Net-(R4-Pad2)
- R50 pad 1: /PWM_TOP_1 -> GND
- R50 pad 2: Net-(C31-Pad2) -> /err_2
- R51 pad 1: /PWM_TOP_1 -> +3.3V
- R51 pad 2: Net-(Q2-B) -> /err_2
- R53 pad 1: Vdrive -> /PWM_TOP_2
- R53 pad 2: /Adequação Sinais Driver/Conectores - PWM e erro/PWM_BOT_int -> /Adequação Sinais Driver/Conectores - PWM e erro1/Adequação Sinais - PWM1/in_sign_aux
- R54 pad 1: Vdrive -> /Adequação Sinais Driver/Conectores - PWM e erro1/Adequação Sinais - PWM1/in_sign_aux
- R54 pad 2: /Adequação Sinais Driver/Conectores - PWM e erro/PWM_BOT_int -> GND
- R56 pad 1: /PWM_TOP_2 -> Vdrive
- R56 pad 2: Net-(Q3-B) -> /Adequação Sinais Driver/Conectores - PWM e erro1/PWM_BOT_int
- R58 pad 1: Vdrive -> /PWM_BOT_2
- R58 pad 2: /Adequação Sinais Driver/Conectores - PWM e erro1/PWM_BOT_int -> /Adequação Sinais Driver/Conectores - PWM e erro1/Adequação Sinais - PWM/in_sign_aux
- R59 pad 1: Vdrive -> /Adequação Sinais Driver/Conectores - PWM e erro1/Adequação Sinais - PWM/in_sign_aux
- R59 pad 2: /Adequação Sinais Driver/Conectores - PWM e erro1/PWM_BOT_int -> GND
- R61 pad 1: /PWM_TOP_3 -> Vdrive
- R61 pad 2: Net-(Q4-B) -> /Adequação Sinais Driver/Conectores - PWM e erro1/PWM_TOP_int
- R62 pad 1: Net-(Q4-B) -> /Adequação Sinais Driver/Conectores - PWM e erro2/erro_driver
- R62 pad 2: GND -> Net-(R62-Pad2)
- R63 pad 1: Vdrive -> /err_3
- R63 pad 2: /Adequação Sinais Driver/Conectores - PWM e erro2/PWM_BOT_int -> /Adequação Sinais Driver/Conectores - PWM e erro2/erro_driver
- R64 pad 1: Vdrive -> GND
- R64 pad 2: /Adequação Sinais Driver/Conectores - PWM e erro2/PWM_BOT_int -> /err_3
- R65 pad 1: /Adequação Sinais Driver/Conectores - PWM e erro1/erro_driver -> +3.3V
- R65 pad 2: Net-(C37-Pad2) -> /err_3
- R67 pad 1: GND -> /PWM_TOP_3
- R67 pad 2: Net-(R66-Pad1) -> /Adequação Sinais Driver/Conectores - PWM e erro2/Adequação Sinais - PWM1/in_sign_aux
- R68 pad 1: +3.3V -> /Adequação Sinais Driver/Conectores - PWM e erro2/Adequação Sinais - PWM1/in_sign_aux
- R68 pad 2: /err_2 -> GND
- R70 pad 1: /PWM_BOT_2 -> Vdrive
- R70 pad 2: Net-(Q5-B) -> /Adequação Sinais Driver/Conectores - PWM e erro2/PWM_BOT_int
- R72 pad 1: Vdrive -> /PWM_BOT_3
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Routing:
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- added copper zone on B.Cu, net GND
- added copper zone on F.Cu, net GND
Other:
- board outline added: 148 x 126 mm

Commit message: Criação dos arquivos em C para o firmware dos dois micros e script em python para salvar aquisição dos dados e envio de comandos
Parts:
- R10, R17, R18, R25, R26, R3, R33, R34, R6, R9: value 91 1/8W -> 100 1/8W
- R49, R63, R77: value 39k -> 12k
- R50, R64, R78: value 11k -> 3k3
- R53, R58, R67, R72, R81, R86: value 180 -> 178
- U8: value TJA1050 -> Módulo TJA1050
Connections:
- C20 pad 1: /PWM_TOP_2 -> /PWM_BOT_2
- C22 pad 1: /PWM_BOT_2 -> /PWM_TOP_2
- C36 pad 1: /PWM_BOT_1 -> /PWM_TOP_1
- C38 pad 1: /PWM_TOP_1 -> /PWM_BOT_1
- R53 pad 1: /PWM_TOP_2 -> /PWM_BOT_2
- R58 pad 1: /PWM_BOT_2 -> /PWM_TOP_2
- R81 pad 1: /PWM_BOT_1 -> /PWM_TOP_1
- R86 pad 1: /PWM_TOP_1 -> /PWM_BOT_1
- U11 pad 3: /PWM_TOP_2 -> /PWM_BOT_2
- U11 pad 5: /PWM_BOT_2 -> /PWM_TOP_2
- U22 pad 33: /PWM_TOP_2 -> /PWM_BOT_2
- U22 pad 34: /PWM_BOT_2 -> /PWM_TOP_2
- U22 pad 36: /PWM_TOP_1 -> /PWM_BOT_1
- U22 pad 37: /PWM_BOT_1 -> /PWM_TOP_1
- U9 pad 3: /PWM_TOP_1 -> /PWM_BOT_1
- U9 pad 5: /PWM_BOT_1 -> /PWM_TOP_1
Routing:
- net /PWM_TOP_2: track 73.7 -> 115.7 mm
- net /PWM_BOT_2: track 115.7 -> 73.7 mm
- net /PWM_TOP_1: track 109.2 -> 147.1 mm
- net /PWM_BOT_1: track 147.1 -> 109.2 mm
